Commit message: Fix directions and finger slider + faster gesture classification

File: frontend/public/models/urdf/arctos_urdf.urdf (robot description, URDF)
Before this commit: robot arctos, 10 links, 9 joints
Joints:
- joint joint2: axis 1.0 -0.0 -0.0 -> -1.0 -0.0 -0.0
- joint joint3: axis -1.0 -0.0 0.0 -> 1.0 -0.0 0.0
- joint joint5: axis -1.0 -0.0 0.0 -> 1.0 -0.0 0.0
