Commit message: Fix joint 6 direction movement

File: backend/models/urdf/arctos_urdf.urdf (robot description, URDF)
Before this commit: robot arctos, 10 links, 9 joints
Joints:
- joint joint2: axis 1.0 -0.0 -0.0 -> -1.0 -0.0 -0.0
- joint joint3: axis -1.0 -0.0 0.0 -> 1.0 -0.0 0.0
- joint joint5: axis -1.0 -0.0 0.0 -> 1.0 -0.0 0.0
- joint joint6: axis -0.0 1.0 -0.0 -> -0.0 -1.0 -0.0

File: frontend/public/models/urdf/arctos_urdf.urdf (robot description, URDF)
Before this commit: robot arctos, 10 links, 9 joints
Joints:
- joint joint6: axis -0.0 1.0 -0.0 -> -0.0 -1.0 -0.0
